File: SPI_Switch.sch (EAGLE design)
At the start: 7 parts

Commit message: updated library parts for easier schematic
Parts:
- added C1: 220uF electrolytic, SparkFun-Passives:CAP0805
- added C2: 47uF, SparkFun-Passives:CAP0805
- added C3: 10uF, SparkFun-Passives:CAP0805
- added C4: 1uF, SparkFun-Passives:CAP0805
- added CE, CLK, DATA, RST: PTR1PAD1-13, testpad:PTR1PAD1-13
- added R1, R2, R3, R4: 0, SparkFun-Passives:RESISTOR0805-RES
Connections:
- removed net N$1: U$3.1, U$7.1
- removed net N$2: U$3.2, U$7.2
- removed net N$3: U$3.3, U$7.3
- new net +24V: C1.1, U$3.1, U$7.1
- new net +5V: C2.1, C3.1, C4.1, U$3.2, U$5.11_VSO, U$5.23_VDD, U$7.2
- new net CE: CE.TP, R4.1, U$1.6, U$4.12_4A
- new net CE_POST: R4.2, U$4.11_4Y
- new net CLK: CLK.TP, R2.1, U$1.2, U$4.5_2A, U$5.13_SCLK
- new net CLK_POST: R2.2, U$4.6_2Y
- new net DATA_IN: DATA.TP, U$1.8, U$5.14_SI
- new net DATA_OUT: R1.1, U$4.2_1A, U$5.12_SO
- new net DATA_OUT_POST: R1.2, U$4.3_1Y
- new net GND: C1.2, C2.2, C3.2, C4.2, U$1.1, U$1.3, U$1.5, U$1.7, U$3.3, U$5.17_GND, U$5.18_GND, U$5.19_GND, U$5.20_GND, U$5.5_GND, U$5.6_GND, U$5.7_GND, U$5.8_GND, U$7.3
- new net RST: R3.1, RST.TP, U$1.4, U$4.9_3A, U$5.24_RST
- new net RST_POST: R3.2, U$4.8_3Y
Other:
- note added: "Power Connectors"
- note added: "Power Filter Capacitors"
- moved on the sheet: U$1, U$2, U$3, U$4, U$5, U$6, U$7

Commit message: added stuff
Parts:
- added C5, C6: 10uF, SparkFun-Passives:CAP0805
- added LED1, LED2, LED3, LED4, LED5, LED6, LED7: (no value), led:LED
- added R10, R11, R12, R6, R7, R8, R9: 1k, SparkFun-Passives:RESISTOR0805-RES
- added R5: DNP, SparkFun-Passives:RESISTOR0805-RES
Connections:
- new net CH1: U$2.3_PATH1, U$2.4_PATH1, U$5.21_OUT0
- new net CH2: U$2.5_PATH2, U$2.6_PATH2, U$5.22_OUT1
- new net CH3: U$2.7_PATH3, U$2.8_PATH3, U$5.3_OUT2
- new net CH4: U$2.10_PATH4, U$2.9_PATH4, U$5.4_OUT3
- new net CH5: U$2.11_PATH5, U$2.12_PATH5, U$5.9_OUT4
- new net CH6: U$2.13_PATH6, U$2.14_PATH6, U$5.10_OUT5
- new net CH7: U$2.16_OPENALL, U$5.15_OUT6
- new net CH8: R5.1, U$5.16_OUT7
- new net N$1: LED1.A, R7.2
- new net N$10: LED5.A, R10.2
- new net N$19: LED6.A, R11.2
- new net N$21: LED7.A, R12.2
- new net N$3: LED2.A, R6.2
- new net N$5: LED3.A, R8.2
- new net N$7: LED4.A, R9.2
- net +24V: now also U$2.1_24VCC
- net +5V: now also C5.1, C6.1, U$4.10_3OE, U$4.13_4OE, U$4.14_VCC, U$4.1_1OE, U$4.4_2OE
- net CE_POST: now also U$6.6
- net CLK_POST: now also U$6.2
- net DATA_OUT_POST: now also U$6.8
- net GND: now also C5.2, C6.2, R5.2, U$2.15_GND, U$4.7_GND, U$6.1, U$6.3, U$6.5, U$6.7
- net RST_POST: now also U$6.4
Other:
- note added: "11/26/2013"
- note added: "Bypass caps for TLE7230G VSO/VDD"
- note added: "Bypassable Line Driver"
- note added: "Input RJ45"
- note added: "Output RJ45"
- note added: "SPI Controlled 8 Channel Switch"
- note added: "SPI Switch Board"
- note added: "Test Points"
- note added: "rev1"
- moved on the sheet: U$2, U$6

Commit message: finished first take
Parts:
- added Q1, Q2, Q3, Q4, Q5, Q6, Q7: MOSFET-NCHANNELBSS123LT1G, SparkFun-DiscreteSemi:MOSFET-NCHANNELBSS123LT1G
- LED1, LED2, LED3, LED4, LED5, LED6: value (none) -> GREEN
- LED7: value (none) -> RED
Connections:
- new net N$10: LED5.C, Q5.D
- new net N$12: LED6.C, Q6.D
- new net N$14: LED7.C, Q7.D
- new net N$2: LED1.C, Q1.D
- new net N$4: LED2.C, Q2.D
- new net N$6: LED3.C, Q3.D
- new net N$8: LED4.C, Q4.D
- net +24V: now also R10.1, R11.1, R12.1, R6.1, R7.1, R8.1, R9.1
- net CH1: now also Q1.G
- net CH2: now also Q2.G
- net CH3: now also Q3.G
- net CH4: now also Q4.G
- net CH5: now also Q5.G
- net CH6: now also Q6.G
- net CH7: now also Q7.G
- net GND: now also Q1.S, Q2.S, Q3.S, Q4.S, Q5.S, Q6.S, Q7.S
Other:
- note added: "LED Driver Circuits"
- note added: "Output Switch Connector"
- moved on the sheet: LED1, LED2, LED3, LED4, LED5, LED6, LED7, R10, R11, R12, R6, R7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
