File: SPI_Switch.sch (EAGLE design)
At the start: 40 parts, among them J1 8516-4500PL, J2 1-406525-1, J3 1-406525-1, J4 0705510037, J5 0705510037, U1 TLE7230G, U2 SN74ABT126

Commit message: redoing layout
Parts:
- added H1, H2, H3, H4: MOUNT-HOLE2.8, holes:MOUNT-HOLE2.8
Other:
- note added: "Mounting Holes"
Changed lines of the file:
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@@
 <part name="GND12" library="supply1" deviceset="GND" device=""/>
 <part name="P+17" library="supply1" deviceset="+24V" device=""/>
-<part name="J1" library="SPI_Switch" deviceset="8516-4500PL" device=""/>
 <part name="C7" library="SparkFun-Passives" deviceset="CAP_POL" device="E" value="220uF"/>
 <part name="P+18" library="supply1" deviceset="+24V" device=""/>
@@
 <part name="R12" library="SparkFun-Passives" deviceset="RESISTOR" device="1206" value="1.5k"/>
 <part name="R13" library="SparkFun-Passives" deviceset="RESISTOR" device="1206" value="1.5k"/>
+<part name="J1" library="SPI_Switch" deviceset="8516-4500PL" device=""/>
+<part name="H1" library="holes" deviceset="MOUNT-HOLE" device="2.8"/>
+<part name="H2" library="holes" deviceset="MOUNT-HOLE" device="2.8"/>
+<part name="H3" library="holes" deviceset="MOUNT-HOLE" device="2.8"/>
+<part name="H4" library="holes" deviceset="MOUNT-HOLE" device="2.8"/>
 </parts>
 <sheets>
@@
 <text x="342.9" y="327.66" size="1.778" layer="91">Output Switch Connector</text>
 <text x="73.66" y="381" size="1.778" layer="91">Power Indication LEDs</text>
+<text x="53.34" y="251.46" size="1.778" layer="91">Mounting Holes</text>
 </plain>
 <instances>
@@
 <instance part="GND12" gate="1" x="124.46" y="274.32"/>
 <instance part="P+17" gate="1" x="299.72" y="335.28"/>
-<instance part="J1" gate="G$1" x="355.6" y="266.7"/>
 <instance part="C7" gate="G$1" x="147.32" y="48.26"/>
 <instance part="P+18" gate="1" x="81.28" y="373.38"/>
@@
 <instance part="R12" gate="G$1" x="284.48" y="325.12" rot="R90"/>
 <instance part="R13" gate="G$1" x="299.72" y="325.12" rot="R90"/>
+<instance part="J1" gate="G$1" x="355.6" y="266.7"/>
+<instance part="H1" gate="G$1" x="58.42" y="238.76"/>
+<instance part="H2" gate="G$1" x="58.42" y="233.68"/>
+<instance part="H3" gate="G$1" x="58.42" y="228.6"/>
+<instance part="H4" gate="G$1" x="58.42" y="223.52"/>
 </instances>
 <busses>
@@
 <wire x1="342.9" y1="297.18" x2="342.9" y2="302.26" width="0.1524" layer="91"/>
 <wire x1="342.9" y1="302.26" x2="350.52" y2="302.26" width="0.1524" layer="91"/>
-<pinref part="J1" gate="G$1" pin="3_PATH1"/>
 <pinref part="LED1" gate="G$1" pin="C"/>
 <wire x1="208.28" y1="309.88" x2="208.28" y2="297.18" width="0.1524" layer="91"/>
 <junction x="208.28" y="297.18"/>
+<pinref part="J1" gate="G$1" pin="3_PATH1"/>
 </segment>
 </net>
@@
 <label x="187.96" y="294.64" size="1.778" layer="95"/>
 <label x="325.12" y="294.64" size="1.778" layer="95"/>
-<pinref part="J1" gate="G$1" pin="5_PATH2"/>
 <pinref part="LED2" gate="G$1" pin="C"/>
 <wire x1="220.98" y1="309.88" x2="220.98" y2="294.64" width="0.1524" layer="91"/>
 <junction x="220.98" y="294.64"/>
+<pinref part="J1" gate="G$1" pin="5_PATH2"/>
 </segment>
 </net>
@@
 <label x="187.96" y="292.1" size="1.778" layer="95"/>
 <label x="325.12" y="292.1" size="1.778" layer="95"/>
-<pinref part="J1" gate="G$1" pin="7_PATH3"/>
 <pinref part="LED3" gate="G$1" pin="C"/>
 <wire x1="233.68" y1="292.1" x2="350.52" y2="292.1" width="0.1524" layer="91"/>
 <wire x1="233.68" y1="309.88" x2="233.68" y2="292.1" width="0.1524" layer="91"/>
 <junction x="233.68" y="292.1"/>
+<pinref part="J1" gate="G$1" pin="7_PATH3"/>
 </segment>
 </net>
@@
 <wire x1="345.44" y1="289.56" x2="345.44" y2="287.02" width="0.1524" layer="91"/>
 <wire x1="345.44" y1="287.02" x2="350.52" y2="287.02" width="0.1524" layer="91"/>
-<pinref part="J1" gate="G$1" pin="9_PATH4"/>
 <pinref part="LED4" gate="G$1" pin="C"/>
 <wire x1="246.38" y1="309.88" x2="246.38" y2="289.56" width="0.1524" layer="91"/>
 <junction x="246.38" y="289.56"/>
+<pinref part="J1" gate="G$1" pin="9_PATH4"/>
 </segment>
 </net>
@@
 <wire x1="342.9" y1="287.02" x2="342.9" y2="281.94" width="0.1524" layer="91"/>
 <wire x1="342.9" y1="281.94" x2="350.52" y2="281.94" width="0.1524" layer="91"/>
-<pinref part="J1" gate="G$1" pin="11_PATH5"/>
 <pinref part="LED5" gate="G$1" pin="C"/>
 <wire x1="259.08" y1="309.88" x2="259.08" y2="287.02" width="0.1524" layer="91"/>
 <junction x="259.08" y="287.02"/>
+<pinref part="J1" gate="G$1" pin="11_PATH5"/>
 </segment>
 </net>
@@
 <wire x1="340.36" y1="284.48" x2="340.36" y2="276.86" width="0.1524" layer="91"/>
 <wire x1="340.36" y1="276.86" x2="350.52" y2="276.86" width="0.1524" layer="91"/>
-<pinref part="J1" gate="G$1" pin="13_PATH6"/>
 <pinref part="LED6" gate="G$1" pin="C"/>
 <wire x1="271.78" y1="309.88" x2="271.78" y2="284.48" width="0.1524" layer="91"/>
 <junction x="271.78" y="284.48"/>
+<pinref part="J1" gate="G$1" pin="13_PATH6"/>
 </segment>
 </net>
@@
 <label x="187.96" y="281.94" size="1.778" layer="95"/>
 <label x="325.12" y="281.94" size="1.778" layer="95"/>
-<pinref part="J1" gate="G$1" pin="16_OPENALL"/>
 <pinref part="LED7" gate="G$1" pin="C"/>
 <wire x1="284.48" y1="309.88" x2="284.48" y2="281.94" width="0.1524" layer="91"/>
 <junction x="284.48" y="281.94"/>
-</segment>
-</net>
+<pinref part="J1" gate="G$1" pin="16_OPENALL"/>
+</segment>
+</net>
